Commit message: Added visualization for imu simulator

File: src/g425_assign4_pkg/include/sim.urdf.xacro (robot description, xacro)
@@ -4,5 +4,5 @@
   <link name="map"/>
   <!-- Cube -->
-  <link name="base_footprint">
+  <link name="mecanum_base_link">
     <visual>
       <origin xyz="0 0 0" rpy="0 0 0"/>
@@ -30,7 +30,38 @@
   </link>
   <!-- Fixed joint from map → cube -->
-  <joint name="map_to_base" type="fixed">
+  <joint name="map_to_mecanum" type="fixed">
     <parent link="map"/>
-    <child link="base_footprint"/>
+    <child link="mecanum_base_link"/>
+    <origin xyz="0 0 0" rpy="0 0 0"/>
+  </joint>
+  <link name="imu_base_link">
+    <visual>
+      <origin xyz="0 0 0" rpy="0 0 0"/>
+      <geometry>
+        <box size="0.3 0.3 0.1"/>
+      </geometry>
+      <material name="green">
+        <color rgba="0 1 0 1"/>
+      </material>
+    </visual>
+    <collision>
+      <origin xyz="0 0 0.5" rpy="0 0 0"/>
+      <geometry>
+        <box size="0.3 0.3 0.1"/>
+      </geometry>
+    </collision>
+    <inertial>
+      <origin xyz="0 0 0" rpy="0 0 0"/>
+      <mass value="1.0"/>
+      <inertia
+        ixx="0.1" ixy="0" ixz="0"
+        iyy="0.1" iyz="0"
+        izz="0.1"/>
+    </inertial>
+  </link>
+  <!-- Fixed joint from map → cube -->
+  <joint name="map_to_imu" type="fixed">
+    <parent link="map"/>
+    <child link="imu_base_link"/>
     <origin xyz="0 0 0" rpy="0 0 0"/>
   </joint>

Commit message: added wheels

File: src/g425_assign4_pkg/include/sim.urdf.xacro (robot description, xacro)
@@ -2,67 +2,134 @@
 <robot name="moving_cube" xmlns:xacro="http://www.ros.org/wiki/xacro">
   <!-- Root frame -->
-  <link name="map"/>
+  <link name="map" />
   <!-- Cube -->
   <link name="mecanum_base_link">
-    <visual>
-      <origin xyz="0 0 0" rpy="0 0 0"/>
-      <geometry>
-        <box size="0.3 0.3 0.1"/>
-      </geometry>
-      <material name="blue">
-        <color rgba="0 0 1 1"/>
-      </material>
-    </visual>
-    <collision>
-      <origin xyz="0 0 0.5" rpy="0 0 0"/>
-      <geometry>
-        <box size="0.3 0.3 0.1"/>
-      </geometry>
-    </collision>
-    <inertial>
-      <origin xyz="0 0 0" rpy="0 0 0"/>
-      <mass value="1.0"/>
-      <inertia
-        ixx="0.1" ixy="0" ixz="0"
-        iyy="0.1" iyz="0"
-        izz="0.1"/>
-    </inertial>
+  <visual>
+    <origin xyz="0 0 0" rpy="0 0 0" />
+    <geometry>
+      <box size="0.3 0.3 0.1" />
+    </geometry>
+    <material name="blue">
+      <color rgba="0 0 1 1" />
+    </material>
+  </visual>
+  <collision>
+    <origin xyz="0 0 0.5" rpy="0 0 0" />
+    <geometry>
+      <box size="0.3 0.3 0.1" />
+    </geometry>
+  </collision>
+  <inertial>
+    <origin xyz="0 0 0" rpy="0 0 0" />
+    <mass value="1.0" />
+    <inertia ixx="0.1" ixy="0" ixz="0" iyy="0.1" iyz="0" izz="0.1" />
+  </inertial>
   </link>
+  <!-- Wheels -->
+  <!-- Front-left wheel -->
+  <link name="wheel_fl">
+  <visual>
+    <origin xyz="0 0 0" rpy="0 0 90" />
+    <geometry>
+      <cylinder radius="0.04" length="0.02" />
+    </geometry>
+    <material name="black">
+      <color rgba="0 0 0 1" />
+    </material>
+  </visual>
+  </link>
+  <joint name="joint_wheel_fl" type="continuous">
+    <parent link="mecanum_base_link" />
+    <child link="wheel_fl" />
+    <origin xyz="0.13 0.16 -0.05" rpy="1.570796327 0 0" />
+    <axis xyz="0 0 1" />
+  </joint>
+  <!-- Front-right wheel -->
+  <link name="wheel_fr">
+  <visual>
+    <origin xyz="0 0 0" rpy="0 0 90" />
+    <geometry>
+      <cylinder radius="0.04" length="0.02" />
+    </geometry>
+    <material name="black">
+      <color rgba="0 0 0 1" />
+    </material>
+  </visual>
+  </link>
+  <joint name="joint_wheel_fr" type="continuous">
+    <parent link="mecanum_base_link" />
+    <child link="wheel_fr" />
+    <origin xyz="0.13 -0.16 -0.05" rpy="-1.570796327 0 0" />
+    <axis xyz="0 0 1" />
+  </joint>
+  <!-- Rear-left wheel -->
+  <link name="wheel_rl">
+  <visual>
+    <origin xyz="0 0 0" rpy="0 0 90" />
+    <geometry>
+      <cylinder radius="0.04" length="0.02" />
+    </geometry>
+    <material name="black">
+      <color rgba="0 0 0 1" />
+    </material>
+  </visual>
+  </link>
+  <joint name="joint_wheel_rl" type="continuous">
+    <parent link="mecanum_base_link" />
+    <child link="wheel_rl" />
+    <origin xyz="-0.13 0.16 -0.05" rpy="1.570796327 0 0" />
+    <axis xyz="0 0 1" />
+  </joint>
+  <!-- Rear-right wheel -->
+  <link name="wheel_rr">
+  <visual>
+    <origin xyz="0 0 0" rpy="0 0 90" />
+    <geometry>
+      <cylinder radius="0.04" length="0.02" />
+    </geometry>
+    <material name="black">
+      <color rgba="0 0 0 1" />
+    </material>
+  </visual>
+  </link>
+  <joint name="joint_wheel_rr" type="continuous">
+    <parent link="mecanum_base_link" />
+    <child link="wheel_rr" />
+    <origin xyz="-0.13 -0.16 -0.05" rpy="-1.570796327 0 0" />
+    <axis xyz="0 0 -1" />
+  </joint>
   <!-- Fixed joint from map → cube -->
   <joint name="map_to_mecanum" type="fixed">
-    <parent link="map"/>
-    <child link="mecanum_base_link"/>
-    <origin xyz="0 0 0" rpy="0 0 0"/>
+    <parent link="map" />
+    <child link="mecanum_base_link" />
+    <origin xyz="0 0 0" rpy="0 0 0" />
   </joint>
   <link name="imu_base_link">
-    <visual>
-      <origin xyz="0 0 0" rpy="0 0 0"/>
-      <geometry>
-        <box size="0.3 0.3 0.1"/>
-      </geometry>
-      <material name="green">
-        <color rgba="0 1 0 1"/>
-      </material>
-    </visual>
-    <collision>
-      <origin xyz="0 0 0.5" rpy="0 0 0"/>
-      <geometry>
-        <box size="0.3 0.3 0.1"/>
-      </geometry>
-    </collision>
-    <inertial>
-      <origin xyz="0 0 0" rpy="0 0 0"/>
-      <mass value="1.0"/>
-      <inertia
-        ixx="0.1" ixy="0" ixz="0"
-        iyy="0.1" iyz="0"
-        izz="0.1"/>
-    </inertial>
+  <visual>
+    <origin xyz="0 0 0" rpy="0 0 0" />
+    <geometry>
+      <box size="0.3 0.3 0.1" />
+    </geometry>
+    <material name="green">
+      <color rgba="0 1 0 1" />
+    </material>
+  </visual>
+  <collision>
+    <origin xyz="0 0 0.5" rpy="0 0 0" />
+    <geometry>
+      <box size="0.3 0.3 0.1" />
+    </geometry>
+  </collision>
+  <inertial>
+    <origin xyz="0 0 0" rpy="0 0 0" />
+    <mass value="1.0" />
+    <inertia ixx="0.1" ixy="0" ixz="0" iyy="0.1" iyz="0" izz="0.1" />
+  </inertial>
   </link>
   <!-- Fixed joint from map → cube -->
   <joint name="map_to_imu" type="fixed">
-    <parent link="map"/>
-    <child link="imu_base_link"/>
-    <origin xyz="0 0 0" rpy="0 0 0"/>
+    <parent link="map" />
+    <child link="imu_base_link" />
+    <origin xyz="0 0 0" rpy="0 0 0" />
   </joint>
 </robot>
